Commit message: feat: STORY-014/015 統合bringup - 設計・テスト・実装（51/51テストパス）
- URDF: imu_link追加（base_link→imu_link TF接続）
- robot_base.launch.py: TF+Motor統合（use_motor条件付き）
- sensors.launch.py: LiDAR+IMU統合（use_lidar/use_imu条件付き）
- zeuscar.launch.py: 全体統合（use_slam/use_rviz条件付き）
- setup.py: launch/configディレクトリ追加
- テスト: test_urdf_imu_link.py(12件)+test_launch_files.py(39件)
- 設計仕様書・実装ガイド・索引更新

Co-Authored-By: Claude Opus 4.6 <noreply@anthropic.com>

File: ros2_ws/src/zeuscar_description/urdf/zeuscar.urdf.xacro (robot description, xacro)
@@ -5,5 +5,6 @@
     base_footprint - 地面投影フレーム（z=0）
       └── base_link - ロボット本体中心
-            └── laser_frame - LiDARスキャン面
+            ├── laser_frame - LiDARスキャン面
+            └── imu_link - IMUセンサー位置
   座標系: REP-103準拠
     X軸: 前方が正
@@ -31,4 +32,9 @@
   <xacro:property name="lidar_radius" value="0.035"/>
   <xacro:property name="lidar_height" value="0.04"/>
+  <!-- IMU取り付け位置 (m) -->
+  <!-- 実測値未計測のため仮値を使用 -->
+  <xacro:property name="imu_x" value="0.0"/>
+  <xacro:property name="imu_y" value="0.0"/>
+  <xacro:property name="imu_z" value="0.05"/>
   <!-- ========== リンク定義 ========== -->
   <!-- base_footprint: 地面投影フレーム -->
@@ -93,3 +99,17 @@
             rpy="0 0 ${lidar_yaw}"/>
   </joint>
+  <!-- base_link → imu_link -->
+  <!--
+    IMU取り付け位置（仮値）:
+    - X: 0mm（本体中心）
+    - Y: 0mm（本体中心）
+    - Z: 50mm（base_linkからの相対高さ）
+    NOTE: 実測値が得られたら更新すること
+  -->
+  <link name="imu_link"/>
+  <joint name="base_link_to_imu" type="fixed">
+    <parent link="base_link"/>
+    <child link="imu_link"/>
+    <origin xyz="${imu_x} ${imu_y} ${imu_z}" rpy="0 0 0"/>
+  </joint>
 </robot>
